File: NomobotSK.kicad_sch (KiCad schematic)
At the start: 72 parts, among them J1 Conn_01x12_Pin, J2 Conn_01x03_Socket, J3 Conn_01x03_Socket, J4 Conn_01x03_Socket, J5 Conn_01x12_Pin, J6 Conn_01x12_Pin, M1 Motor_DC, M2 Motor_DC, SW1 SW_DIP_x01, SW2 SW_Push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

Commit message: change design of comparator
Parts:
- added R12, R13: 1K, Resistor_SMD:R_0805_2012Metric, symbol Device:R_US
- R10, R11: value 1K -> 330R
Connections:
- net 3V3: now also R12.1, R13.2
- net LIN_L: now also R13.1
- net LIN_R: now also R12.2

Commit message: routing done
Parts:
- removed A1: NodeMCU V2 Amica, NodeMCU V2 AMICA:NodeMCU V2 Amica, symbol NodeMCU V2 AMICA:NodeMCU V2 Amica
- removed BT1: BH-18650-PC, BH-18650-PC:BAT_BH-18650-PC, symbol BH-18650-PC:BH-18650-PC
- removed BZ1: Buzzer, Buzzer_Beeper:Buzzer_12x9.5RM7.6, symbol Device:Buzzer
- removed C1, C8: 1u, Capacitor_SMD:C_0805_2012Metric, symbol Device:C
- removed C10, C7: C_Polarized, Capacitor_SMD:CP_Elec_6.3x5.3, symbol Device:C_Polarized
- removed C2, C3, C4, C5, C6: 100n, Capacitor_SMD:C_0805_2012Metric, symbol Device:C
- removed D1, D10, D11, D12, D13, D14, D15, D16, D2, D3, D4, D5, D6, D7, D8, D9: WS2812B, LED_SMD:LED_WS2812B_PLCC4_5.0x5.0mm_P3.2mm, symbol LED:WS2812B
- removed D17, D18: LED_Green, LED_SMD:LED_0805_2012Metric, symbol Device:LED
- removed J1, J5, J6: Conn_01x12_Pin, Connector_PinHeader_2.54mm:PinHeader_1x12_P2.54mm_Vertical, symbol Connector:Conn_01x12_Pin
- removed J2, J3, J4: Conn_01x03_Socket, Connector_JST:JST_EH_B3B-EH-A_1x03_P2.50mm_Vertical, symbol Connector:Conn_01x03_Socket
- removed M1, M2: Motor_DC, TerminalBlock_TE-Connectivity:TerminalBlock_TE_282834-2_1x02_P2.54mm_Horizontal, symbol Motor:Motor_DC
- removed R1: 470R, Resistor_SMD:R_0805_2012Metric, symbol Device:R_US
- removed R10, R11: 330R, Resistor_SMD:R_0805_2012Metric, symbol Device:R_US
- removed R12, R13: 1K, Resistor_SMD:R_0805_2012Metric, symbol Device:R_US
- removed R2, R3: 220R, Resistor_SMD:R_0805_2012Metric, symbol Device:R_US
- removed R4, R5, R6, R7, R8: 10K, Resistor_SMD:R_0805_2012Metric, symbol Device:R_US
- removed R9: 100R, Resistor_SMD:R_0805_2012Metric, symbol Device:R_US
- removed RV1, RV2: Trimpot_10K, Potentiometer_THT:Potentiometer_Runtron_RM-065_Vertical, symbol Device:R_Potentiometer_Trim_US
- removed SW1: SW_DIP_x01, Button_Switch_THT:SW_DIP_SPSTx01_Slide_9.78x4.72mm_W7.62mm_P2.54mm, symbol Switch:SW_DIP_x01
- removed SW2, SW3, SW4: SW_Push, Button_Switch_THT:SW_PUSH_6mm_H4.3mm, symbol Switch:SW_Push
- removed SW5: SW_DIP_x10, Button_Switch_THT:SW_DIP_SPSTx10_Slide_9.78x27.58mm_W7.62mm_P2.54mm, symbol Switch:SW_DIP_x10
- removed SW6: SW_DIP_x04, Button_Switch_THT:SW_DIP_SPSTx04_Slide_9.78x12.34mm_W7.62mm_P2.54mm, symbol Switch:SW_DIP_x04
- removed TP1: LED_TP, TestPoint:TestPoint_Pad_D1.0mm, symbol Connector:TestPoint
- removed TP2: 3v3, TestPoint:TestPoint_Pad_D2.0mm, symbol Connector:TestPoint
- removed TP3, TP4, TP5, TP6, TP7, TP8: TestPoint, TestPoint:TestPoint_Pad_D1.0mm, symbol Connector:TestPoint
- removed U1: L293D, Package_DIP:DIP-16_W7.62mm, symbol Driver_Motor:L293D
- removed U2: TP4056 Module, Modules:TP4056_Module, symbol Modules:TP4056_Module
- removed U3, U4: TCRT5000, TCRT5000:OPTO_TCRT5000, symbol TCRT5000:TCRT5000
- removed U5: HC-SR04, HC-SR04:XCVR_HC-SR04, symbol HC-SR04:HC-SR04
- removed U6: AMS1117-3.3, Package_TO_SOT_SMD:SOT-223-3_TabPin2, symbol Regulator_Linear:AMS1117-3.3
- removed U7: LM393D, LM393D:SOIC127P599X175-8N, symbol LM393D:LM393D
Other:
- added sheet CONNECTOR (Conn_Interface.kicad_sch)
- added sheet LINE SENSOR (Line_Sensor.kicad_sch)
- added sheet MAIN MCU (Main_MCU.kicad_sch)
- added sheet MOTOR (Motor_Driver.kicad_sch)
- added sheet PERIPHERAL (Sensors.kicad_sch)
- added sheet POWER (Power_Circuit.kicad_sch)
- added sheet RGB LED (RGB_Led.kicad_sch)
